File: ESP32DevKitV1.kicad_sch (KiCad schematic)
At the start: 0 parts

Commit message: major changes are done before panalizing
Parts:
- added J2, J5: ESPheader, Connector_PinHeader_2.54mm:PinHeader_1x15_P2.54mm_Vertical, symbol Connector_Generic:Conn_01x15
Connections:
- new net 3V3: J5.15 (Pin_15)
- new net D1: J5.3 (Pin_3)
- new net D12: J2.12 (Pin_12)
- new net D13: J2.13 (Pin_13)
- new net D14: J2.11 (Pin_11)
- new net D15: J5.13 (Pin_13)
- new net D16: J5.10 (Pin_10)
- new net D17: J5.9 (Pin_9)
- new net D18: J5.7 (Pin_7)
- new net D19: J5.6 (Pin_6)
- new net D2: J5.12 (Pin_12)
- new net D21: J5.5 (Pin_5)
- new net D22: J5.2 (Pin_2)
- new net D23: J5.1 (Pin_1)
- new net D25: J2.8 (Pin_8)
- new net D26: J2.9 (Pin_9)
- new net D27: J2.10 (Pin_10)
- new net D3: J5.4 (Pin_4)
- new net D32: J2.6 (Pin_6)
- new net D33: J2.7 (Pin_7)
- new net D34: J2.4 (Pin_4)
- new net D35: J2.5 (Pin_5)
- new net D36: J2.2 (Pin_2)
- new net D39: J2.3 (Pin_3)
- new net D4: J5.11 (Pin_11)
- new net D5: J5.8 (Pin_8)
- new net EN: J2.1 (Pin_1)
- new net EVIN: J2.15 (Pin_15)
- new net GND: J2.14 (Pin_14), J5.14 (Pin_14)
Changed lines of the file:
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@@
-(kicad_sch (version 20211123) (generator eeschema)
+(kicad_sch (version 20230121) (generator eeschema)
   (paper "A4")
+  (hierarchical_label "D14" (shape input) (at 124.46 99.06 180) (fields_autoplaced)
+    (effects (font (size 1.27 1.27)) (justify right))
+  )
+  (hierarchical_label "GND" (shape input) (at 146.05 106.68 0) (fields_autoplaced)
+    (effects (font (size 1.27 1.27)) (justify left))
+  )
+  (hierarchical_label "D15" (shape input) (at 146.05 104.14 0) (fields_autoplaced)
+    (effects (font (size 1.27 1.27)) (justify left))
+  )
+  (hierarchical_label "D4" (shape input) (at 146.05 99.06 0) (fields_autoplaced)
+    (effects (font (size 1.27 1.27)) (justify left))
+  )
+  (hierarchical_label "D17" (shape input) (at 146.05 93.98 0) (fields_autoplaced)
+    (effects (font (size 1.27 1.27)) (justify left))
+  )
+  (hierarchical_label "EVIN" (shape input) (at 124.46 109.22 180) (fields_autoplaced)
+    (effects (font (size 1.27 1.27)) (justify right))
+  )
+  (hierarchical_label "D19" (shape input) (at 146.05 86.36 0) (fields_autoplaced)
+    (effects (font (size 1.27 1.27)) (justify left))
+  )
+  (hierarchical_label "D23" (shape input) (at 146.05 73.66 0) (fields_autoplaced)
+    (effects (font (size 1.27 1.27)) (justify left))
+  )
+  (hierarchical_label "D35" (shape input) (at 124.46 83.82 180) (fields_autoplaced)
+    (effects (font (size 1.27 1.27)) (justify right))
+  )
+  (hierarchical_label "D18" (shape input) (at 146.05 88.9 0) (fields_autoplaced)
+    (effects (font (size 1.27 1.27)) (justify left))
+  )
+  (hierarchical_label "D25" (shape input) (at 124.46 91.44 180) (fields_autoplaced)
+    (effects (font (size 1.27 1.27)) (justify right))
+  )
+  (hierarchical_label "D1" (shape input) (at 146.05 78.74 0) (fields_autoplaced)
+    (effects (font (size 1.27 1.27)) (justify left))
+  )
+  (hierarchical_label "D16" (shape input) (at 146.05 96.52 0) (fields_autoplaced)
+    (effects (font (size 1.27 1.27)) (justify left))
+  )
+  (hierarchical_label "3V3" (shape input) (at 146.05 109.22 0) (fields_autoplaced)
+    (effects (font (size 1.27 1.27)) (justify left))
+  )
+  (hierarchical_label "D13" (shape input) (at 124.46 104.14 180) (fields_autoplaced)
+    (effects (font (size 1.27 1.27)) (justify right))
+  )
+  (hierarchical_label "D33" (shape input) (at 124.46 88.9 180) (fields_autoplaced)
+    (effects (font (size 1.27 1.27)) (justify right))
+  )
+  (hierarchical_label "D39" (shape input) (at 124.46 78.74 180) (fields_autoplaced)
+    (effects (font (size 1.27 1.27)) (justify right))
+  )
+  (hierarchical_label "D36" (shape input) (at 124.46 76.2 180) (fields_autoplaced)
+    (effects (font (size 1.27 1.27)) (justify right))
+  )
+  (hierarchical_label "EN" (shape input) (at 124.46 73.66 180) (fields_autoplaced)
+    (effects (font (size 1.27 1.27)) (justify right))
+  )
+  (hierarchical_label "D26" (shape input) (at 124.46 93.98 180) (fields_autoplaced)
+    (effects (font (size 1.27 1.27)) (justify right))
+  )
+  (hierarchical_label "D5" (shape input) (at 146.05 91.44 0) (fields_autoplaced)
+    (effects (font (size 1.27 1.27)) (justify left))
+  )
+  (hierarchical_label "D27" (shape input) (at 124.46 96.52 180) (fields_autoplaced)
+    (effects (font (size 1.27 1.27)) (justify right))
+  )
+  (hierarchical_label "D21" (shape input) (at 146.05 83.82 0) (fields_autoplaced)
+    (effects (font (size 1.27 1.27)) (justify left))
+  )
+  (hierarchical_label "D22" (shape input) (at 146.05 76.2 0) (fields_autoplaced)
+    (effects (font (size 1.27 1.27)) (justify left))
+  )
+  (hierarchical_label "D3" (shape input) (at 146.05 81.28 0) (fields_autoplaced)
+    (effects (font (size 1.27 1.27)) (justify left))
+  )
+  (hierarchical_label "D2" (shape input) (at 146.05 101.6 0) (fields_autoplaced)
+    (effects (font (size 1.27 1.27)) (justify left))
+  )
+  (hierarchical_label "D34" (shape input) (at 124.46 81.28 180) (fields_autoplaced)
+    (effects (font (size 1.27 1.27)) (justify right))
+  )
+  (hierarchical_label "GND" (shape input) (at 124.46 106.68 180) (fields_autoplaced)
+    (effects (font (size 1.27 1.27)) (justify right))
+  )
+  (hierarchical_label "D12" (shape input) (at 124.46 101.6 180) (fields_autoplaced)
+    (effects (font (size 1.27 1.27)) (justify right))
+  )
+  (hierarchical_label "D32" (shape input) (at 124.46 86.36 180) (fields_autoplaced)
+    (effects (font (size 1.27 1.27)) (justify right))
+  )
+  (symbol (lib_id "Connector_Generic:Conn_01x15") (at 129.54 91.44 0) (unit 1)
+    (in_bom yes) (on_board yes) (dnp no)
+    (property "Reference" "J2" (at 128.27 68.58 0)
+      (effects (font (size 1.27 1.27)) (justify left))
+    )
+    (property "Value" "ESPheader" (at 115.57 68.58 0)
+      (effects (font (size 1.27 1.27)) (justify left))
+    )
+    (property "Footprint" "Connector_PinHeader_2.54mm:PinHeader_1x15_P2.54mm_Vertical" (at 129.54 91.44 0)
+      (effects (font (size 1.27 1.27)) hide)
+    )
+    (property "Datasheet" "https://www.lcsc.com/product-detail/Female-Headers_HCTL-HCTL-PM254-1-15-Z-8.5_C2897378.html" (at 129.54 91.44 0)
+      (effects (font (size 1.27 1.27)) hide)
+    )
+    (property "LCSC" "C2897378" (at 129.54 91.44 0)
+      (effects (font (size 1.27 1.27)) hide)
+    )
+    (pin "1")
+    (pin "10")
+    (pin "11")
+    (pin "12")
+    (pin "13")
+    (pin "14")
+    (pin "15")
+    (pin "2")
+    (pin "3")
+    (pin "4")
+    (pin "5")
+    (pin "6")
+    (pin "7")
+    (pin "8")
+    (pin "9")
+    (instances
+      (project "NoU2"
+        (path "/e83aa78a-7ee8-4825-a22a-a2646798082a/00000000-0000-0000-0000-00006057e9b9"
+          (reference "J2") (unit 1)
+        )
+      )
+    )
+  )
+  (symbol (lib_id "Connector_Generic:Conn_01x15") (at 140.97 91.44 0) (mirror y) (unit 1)
+    (in_bom yes) (on_board yes) (dnp no)
+    (property "Reference" "J5" (at 142.24 68.58 0)
+      (effects (font (size 1.27 1.27)) (justify left))
+    )
+    (property "Value" "ESPheader" (at 154.94 68.58 0)
+      (effects (font (size 1.27 1.27)) (justify left))
+    )
+    (property "Footprint" "Connector_PinHeader_2.54mm:PinHeader_1x15_P2.54mm_Vertical" (at 140.97 91.44 0)
+      (effects (font (size 1.27 1.27)) hide)
+    )
+    (property "Datasheet" "https://www.lcsc.com/product-detail/Female-Headers_HCTL-HCTL-PM254-1-15-Z-8.5_C2897378.html" (at 140.97 91.44 0)
+      (effects (font (size 1.27 1.27)) hide)
+    )
+    (property "LCSC" "C2897378" (at 140.97 91.44 0)
+      (effects (font (size 1.27 1.27)) hide)
+    )
+    (pin "1")
+    (pin "10")
+    (pin "11")
+    (pin "12")
+    (pin "13")
+    (pin "14")
+    (pin "15")
+    (pin "2")
+    (pin "3")
+    (pin "4")
+    (pin "5")
+    (pin "6")
+    (pin "7")
+    (pin "8")
+    (pin "9")
+    (instances
+      (project "NoU2"
+        (path "/e83aa78a-7ee8-4825-a22a-a2646798082a/00000000-0000-0000-0000-00006057e9b9"
+          (reference "J5") (unit 1)
+        )
+      )
+    )
+  )
 )
